File: kicad/GluecksraD.kicad_pcb (KiCad board)
At the start: 2 copper layers, 68 x 68 mm, 27 parts, among them U2 NE555, U3 CD4017

Commit message: V1.2 02.04.2024
Other:
- board text added: "JLCJLCJLCJLC"
